Commit message: Tekerleklere dönüşü gösteren görsel işaret eklendi
Düz silindir tekerleğin kendi ekseni etrafında dönmesi görsel olarak fark edilmiyordu. Her tekerleğin dış yüzüne yalnızca görsel amaçlı gri bir şerit eklendi

File: src/serabot_description/urdf/serabot.urdf.xacro (robot description, xacro)
@@ -78,4 +78,10 @@
         <material name="black"/>
       </visual>
+      <!-- Dış yüzdeki gri şerit: tekerleğin döndüğü gözle görülebilsin -->
+      <visual>
+        <origin xyz="0 ${y_sign*(wheel_width/2 + 0.001)} 0" rpy="0 0 0"/>
+        <geometry><box size="${1.6*wheel_radius} 0.002 0.015"/></geometry>
+        <material name="grey"/>
+      </visual>
       <collision>
         <origin xyz="0 0 0" rpy="${-pi/2} 0 0"/>
